File: prueba/prueba.kicad_pcb (KiCad board)
At the start: 2 copper layers, 60.3 x 58.6 mm, 4 parts, among them J2 Barrel_Jack_MountingPin, U1 mpu6050, U2 LM78L05_TO92

Commit message: eles
Other:
- board size 60.3 x 58.6 mm -> 52 x 73.8 mm
Changed lines of the file:
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@@
 	)
 	(gr_rect
-		(start 18.39 39.91)
-		(end 78.72 98.51)
+		(start 24.56 24.76)
+		(end 76.52 98.51)
 		(stroke
 			(width 0.05)
@@
 		(polygon
 			(pts
-				(xy 18.38 39.9) (xy 79.2 40.13) (xy 78.74 98.53) (xy 18.37 98.51)
+				(xy 24.28 16.47) (xy 80.47 21.5) (xy 78.74 98.53) (xy 18.37 98.51)
 			)
 		)
