File: prueba/prueba.kicad_sch (KiCad schematic)
At the start: 0 parts

Commit message: first
Parts:
- added A1: RaspberryPi_Pico, Module:RaspberryPi_Pico_Common_Unspecified, symbol MCU_Module:RaspberryPi_Pico
- added J2: Barrel_Jack_MountingPin, Connector_BarrelJack:BarrelJack_GCT_DCJ200-10-A_Horizontal, symbol Connector:Barrel_Jack_MountingPin
- added U1: mpu6050, sensors:module_mpu6050, symbol module_mpu6050:module_mpu6050
- added U2: LM78L05_TO92, Package_TO_SOT_THT:TO-92, symbol Regulator_Linear:LM78L05_TO92
Connections:
- new net: J2.2, U2.3 (VI)
- new net CSL: A1.7 (GPIO5), U1.3 (SCL)
- new net SDA: A1.6 (GPIO4), U1.4 (SDA)
- new net gnd: A1.13 (GND), A1.18 (GND), A1.23 (GND), A1.28 (GND), A1.3 (GND), A1.38 (GND), A1.8 (GND), J2.1, U1.2 (GND), U2.2 (GND)
- new net vcc: A1.36 (3V3), U1.1 (VCC), U2.1 (VO)

Commit message: topi
Parts:
- added A2: Arduino_Nano_RP2040_Connect, Module:Arduino_Nano, symbol MCU_Module:Arduino_Nano_RP2040_Connect
Connections:
- net gnd: now also A2.29 (GND), A2.4 (GND)
Changed lines of the file:
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@@
+		)
+	)
+	(global_label "gnd"
+		(shape input)
+		(at 121.92 151.13 270)
+		(fields_autoplaced yes)
+		(effects
+			(font
+				(size 1.27 1.27)
+			)
+			(justify right)
+		)
+		(property "Intersheetrefs" "${INTERSHEET_REFS}"
+			(at 121.92 157.5622 90)
+			(effects
+				(font
+					(size 1.27 1.27)
+				)
+				(justify right)
+				(hide yes)
+			)
 		)
 	)
@@
 					(unit 1)
 				)
+			)
+		)
+	)
+	(symbol
+		(lib_id "MCU_Module:Arduino_Nano_RP2040_Connect")
+		(at 121.92 125.73 0)
+		(unit 1)
+		(exclude_from_sim no)
+		(in_bom yes)
+		(on_board yes)
+		(dnp no)
+		(fields_autoplaced yes)
+		(property "Reference" "A2"
+			(at 121.92 97.79 0)
+			(effects
+				(font
+					(size 1.27 1.27)
+				)
+			)
+		)
+		(property "Value" "Arduino_Nano_RP2040_Connect"
+			(at 121.92 100.33 0)
+			(effects
+				(font
+					(size 1.27 1.27)
+				)
+			)
+		)
+		(property "Footprint" "Module:Arduino_Nano"
+			(at 135.636 159.766 0)
+			(effects
+				(font
+					(size 1.27 1.27)
+					(italic yes)
+				)
+				(hide yes)
+			)
+		)
+		(property "Datasheet" "https://docs.arduino.cc/resources/datasheets/ABX00053-datasheet.pdf"
+			(at 161.036 157.226 0)
+			(effects
+				(font
+					(size 1.27 1.27)
+				)
+				(hide yes)
+			)
+		)
+		(property "Description" "Arduino Nano board based on the RP2040 microcontroller with a dual-core 133 MHz ARM Cortex-M0+ processor, 264 kB SRAM, and up to 16 MB flash memory. Operates at 3.3V, with 5V Micro USB input and 4-20V VIN. Features Wi-Fi®, Bluetooth® LE, digital and analog pins, and supports SPI, I2C, UART, and PIO. Includes a 6-axis IMU, RGB LED, microphone, and cryptographic chip for secure communication."
+			(at 330.962 154.686 0)
+			(effects
+				(font
+					(size 1.27 1.27)
+				)
+				(hide yes)
+			)
+		)
+		(pin "28"
+		)
+		(pin "19"
+		)
+		(pin "24"
+		)
+		(pin "23"
+		)
+		(pin "25"
+		)
+		(pin "21"
+		)
+		(pin "20"
+		)
+		(pin "22"
+		)
+		(pin "26"
+		)
+		(pin "10"
+		)
+		(pin "13"
+		)
+		(pin "14"
+		)
+		(pin "17"
+		)
+		(pin "27"
+		)
+		(pin "29"
+		)
+		(pin "18"
+		)
+		(pin "3"
+		)
+		(pin "9"
+		)
+		(pin "15"
+		)
+		(pin "30"
+		)
+		(pin "8"
+		)
+		(pin "5"
+		)
+		(pin "2"
+		)
+		(pin "6"
+		)
+		(pin "16"
+		)
+		(pin "4"
+		)
+		(pin "1"
+		)
+		(pin "11"
+		)
+		(pin "7"
+		)
+		(pin "12"
+		)
+		(instances
+			(project ""
+				(path "/27c57ad6-5ae0-4715-b811-ded17724261b"
+					(reference "A2")
+					(unit 1)
+				)

Commit message: prueba random
Connections:
- net CSL: now also A2.24 (SCL/A5)
- net SDA: now also A2.23 (SDA/A4)
- net vcc: now also A2.30 (VIN)
- net at A2.1 (D1/TX): now also A2.5 (D2), A2.6 (D3), A2.7 (D4), A2.8 (D5)
Changed lines of the file:
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@@
 	(generator_version "9.0")
 	(paper "A4")
+	(junction
+		(at 101.6 118.11)
+		(diameter 0)
+		(color 0 0 0 0)
+	)
+	(junction
+		(at 101.6 115.57)
+		(diameter 0)
+		(color 0 0 0 0)
+	)
+	(junction
+		(at 101.6 120.65)
+		(diameter 0)
+		(color 0 0 0 0)
+	)
+	(wire
+		(pts
+			(xy 101.6 115.57) (xy 104.14 115.57)
+		)
+		(stroke
+			(width 0)
+			(type default)
+		)
+	)
+	(wire
+		(pts
+			(xy 104.14 120.65) (xy 101.6 120.65)
+		)
+		(stroke
+			(width 0)
+			(type default)
+		)
+	)
+	(wire
+		(pts
+			(xy 101.6 113.03) (xy 101.6 115.57)
+		)
+		(stroke
+			(width 0)
+			(type default)
+		)
+	)
 	(wire
 		(pts
@@
 	(wire
 		(pts
+			(xy 101.6 120.65) (xy 101.6 118.11)
+		)
+		(stroke
+			(width 0)
+			(type default)
+		)
+	)
+	(wire
+		(pts
+			(xy 104.14 113.03) (xy 101.6 113.03)
+		)
+		(stroke
+			(width 0)
+			(type default)
+		)
+	)
+	(wire
+		(pts
 			(xy 142.24 49.53) (xy 143.51 49.53)
 		)
@@
 	(wire
 		(pts
+			(xy 104.14 118.11) (xy 101.6 118.11)
+		)
+		(stroke
+			(width 0)
+			(type default)
+		)
+	)
+	(wire
+		(pts
+			(xy 101.6 118.11) (xy 101.6 115.57)
+		)
+		(stroke
+			(width 0)
+			(type default)
+		)
+	)
+	(wire
+		(pts
+			(xy 101.6 120.65) (xy 101.6 123.19)
+		)
+		(stroke
+			(width 0)
+			(type default)
+		)
+	)
+	(wire
+		(pts
 			(xy 217.17 21.59) (xy 224.79 21.59)
 		)
@@
 	(wire
 		(pts
+			(xy 104.14 123.19) (xy 101.6 123.19)
+		)
+		(stroke
+			(width 0)
+			(type default)
+		)
+	)
+	(wire
+		(pts
 			(xy 209.55 31.75) (xy 209.55 29.21)
 		)
@@
 		)
 	)
+	(global_label "CSL"
+		(shape input)
+		(at 139.7 138.43 0)
+		(fields_autoplaced yes)
+		(effects
+			(font
+				(size 1.27 1.27)
+			)
+			(justify left)
+		)
+		(property "Intersheetrefs" "${INTERSHEET_REFS}"
+			(at 146.1928 138.43 0)
+			(effects
+				(font
+					(size 1.27 1.27)
+				)
+				(justify left)
+				(hide yes)
+			)
+		)
+	)
 	(global_label "SDA"
 		(shape input)
@@
 	(global_label "SDA"
 		(shape input)
+		(at 139.7 135.89 0)
+		(fields_autoplaced yes)
+		(effects
+			(font
+				(size 1.27 1.27)
+			)
+			(justify left)
+		)
+		(property "Intersheetrefs" "${INTERSHEET_REFS}"
+			(at 146.2533 135.89 0)
+			(effects
+				(font
+					(size 1.27 1.27)
+				)
+				(justify left)
+				(hide yes)
+			)
+		)
+	)
+	(global_label "SDA"
+		(shape input)
 		(at 101.6 44.45 180)
 		(fields_autoplaced yes)
@@
 			(effects
 				(font
+					(size 1.27 1.27)
+				)
+				(justify right)
+				(hide yes)
+			)
+		)
+	)
+	(global_label "vcc"
+		(shape input)
+		(at 104.14 105.41 180)
+		(fields_autoplaced yes)
+		(effects
+			(font
+				(size 1.27 1.27)
+			)
+			(justify right)
+		)
+		(property "Intersheetrefs" "${INTERSHEET_REFS}"
+			(at 98.01 105.41 0)
+			(effects
+				(font
