File: prueba/prueba.kicad_sch (KiCad schematic)
At the start: 5 parts, among them J2 Barrel_Jack_MountingPin, U1 mpu6050, U2 LM78L05_TO92

Commit message: eles2
Connections:
- net at A2.1 (D1/TX): now also A2.10 (D7), A2.11 (D8), A2.12 (D9), A2.13 (D10/CS), A2.5 (D2), A2.6 (D3), A2.7 (D4), A2.8 (D5), A2.9 (D6)
- net at A2.2 (D0/RX): now also A2.30 (VIN)
Changed lines of the file:
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@@
 	(generator_version "9.0")
 	(paper "A4")
+	(junction
+		(at 104.14 125.73)
+		(diameter 0)
+		(color 0 0 0 0)
+	)
+	(junction
+		(at 104.14 118.11)
+		(diameter 0)
+		(color 0 0 0 0)
+	)
+	(junction
+		(at 104.14 115.57)
+		(diameter 0)
+		(color 0 0 0 0)
+	)
+	(junction
+		(at 104.14 130.81)
+		(diameter 0)
+		(color 0 0 0 0)
+	)
+	(junction
+		(at 104.14 133.35)
+		(diameter 0)
+		(color 0 0 0 0)
+	)
+	(junction
+		(at 104.14 120.65)
+		(diameter 0)
+		(color 0 0 0 0)
+	)
+	(junction
+		(at 104.14 123.19)
+		(diameter 0)
+		(color 0 0 0 0)
+	)
+	(junction
+		(at 104.14 128.27)
+		(diameter 0)
+		(color 0 0 0 0)
+	)
+	(wire
+		(pts
+			(xy 104.14 133.35) (xy 104.14 135.89)
+		)
+		(stroke
+			(width 0)
+			(type default)
+		)
+	)
+	(wire
+		(pts
+			(xy 104.14 130.81) (xy 104.14 133.35)
+		)
+		(stroke
+			(width 0)
+			(type default)
+		)
+	)
+	(wire
+		(pts
+			(xy 104.14 125.73) (xy 104.14 128.27)
+		)
+		(stroke
+			(width 0)
+			(type default)
+		)
+	)
+	(wire
+		(pts
+			(xy 104.14 105.41) (xy 104.14 110.49)
+		)
+		(stroke
+			(width 0)
+			(type default)
+		)
+	)
 	(wire
 		(pts
@@
 	(wire
 		(pts
+			(xy 104.14 115.57) (xy 104.14 118.11)
+		)
+		(stroke
+			(width 0)
+			(type default)
+		)
+	)
+	(wire
+		(pts
 			(xy 209.55 31.75) (xy 224.79 31.75)
 		)
 		(stroke
+			(width 0)
+			(type default)
+		)
+	)
+	(wire
+		(pts
+			(xy 104.14 120.65) (xy 104.14 123.19)
+		)
+		(stroke
+			(width 0)
+			(type default)
+		)
+	)
+	(wire
+		(pts
+			(xy 104.14 118.11) (xy 104.14 120.65)
+		)
+		(stroke
+			(width 0)
+			(type default)
+		)
+	)
+	(wire
+		(pts
+			(xy 104.14 113.03) (xy 104.14 115.57)
+		)
+		(stroke
+			(width 0)
+			(type default)
+		)
+	)
+	(wire
+		(pts
+			(xy 104.14 123.19) (xy 104.14 125.73)
+		)
+		(stroke
+			(width 0)
+			(type default)
+		)
+	)
+	(wire
+		(pts
+			(xy 104.14 128.27) (xy 104.14 130.81)
+		)
+		(stroke

Commit message: parael emi jaj
Other:
- note added: "EL QUE LO LEA ES GAY"
- moved on the sheet: A2
Changed lines of the file:
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@@
 	(generator_version "9.0")
 	(paper "A4")
+	(text "EL QUE LO LEA ES GAY"
+		(exclude_from_sim no)
+		(at 173.228 110.236 0)
+		(effects
+			(font
+				(size 25.4 25.4)
+			)
+		)
+	)
 	(junction
-		(at 104.14 125.73)
+		(at 113.03 168.91)
 		(diameter 0)
 		(color 0 0 0 0)
 	)
 	(junction
-		(at 104.14 118.11)
+		(at 113.03 161.29)
 		(diameter 0)
 		(color 0 0 0 0)
 	)
 	(junction
-		(at 104.14 115.57)
+		(at 113.03 158.75)
 		(diameter 0)
 		(color 0 0 0 0)
 	)
 	(junction
-		(at 104.14 130.81)
+		(at 113.03 173.99)
 		(diameter 0)
 		(color 0 0 0 0)
 	)
 	(junction
-		(at 104.14 133.35)
+		(at 113.03 176.53)
 		(diameter 0)
 		(color 0 0 0 0)
 	)
 	(junction
-		(at 104.14 120.65)
+		(at 113.03 163.83)
 		(diameter 0)
 		(color 0 0 0 0)
 	)
 	(junction
-		(at 104.14 123.19)
+		(at 113.03 166.37)
 		(diameter 0)
 		(color 0 0 0 0)
 	)
 	(junction
-		(at 104.14 128.27)
+		(at 113.03 171.45)
 		(diameter 0)
 		(color 0 0 0 0)
@@
 	(wire
 		(pts
-			(xy 104.14 133.35) (xy 104.14 135.89)
-		)
-		(stroke
-			(width 0)
-			(type default)
-		)
-	)
-	(wire
-		(pts
-			(xy 104.14 130.81) (xy 104.14 133.35)
-		)
-		(stroke
-			(width 0)
-			(type default)
-		)
-	)
-	(wire
-		(pts
-			(xy 104.14 125.73) (xy 104.14 128.27)
-		)
-		(stroke
-			(width 0)
-			(type default)
-		)
-	)
-	(wire
-		(pts
-			(xy 104.14 105.41) (xy 104.14 110.49)
+			(xy 113.03 176.53) (xy 113.03 179.07)
+		)
+		(stroke
+			(width 0)
+			(type default)
+		)
+	)
+	(wire
+		(pts
+			(xy 113.03 173.99) (xy 113.03 176.53)
+		)
+		(stroke
+			(width 0)
+			(type default)
+		)
+	)
+	(wire
+		(pts
+			(xy 113.03 168.91) (xy 113.03 171.45)
+		)
+		(stroke
+			(width 0)
+			(type default)
+		)
+	)
+	(wire
+		(pts
+			(xy 113.03 148.59) (xy 113.03 153.67)
 		)
 		(stroke
@@
 	(wire
 		(pts
-			(xy 104.14 115.57) (xy 104.14 118.11)
+			(xy 113.03 158.75) (xy 113.03 161.29)
 		)
 		(stroke
@@
 	(wire
 		(pts
-			(xy 104.14 120.65) (xy 104.14 123.19)
-		)
-		(stroke
-			(width 0)
-			(type default)
-		)
-	)
-	(wire
-		(pts
-			(xy 104.14 118.11) (xy 104.14 120.65)
-		)
-		(stroke
-			(width 0)
-			(type default)
-		)
-	)
-	(wire
-		(pts
-			(xy 104.14 113.03) (xy 104.14 115.57)
-		)
-		(stroke
-			(width 0)
-			(type default)
-		)
-	)
-	(wire
-		(pts
-			(xy 104.14 123.19) (xy 104.14 125.73)
-		)
-		(stroke
-			(width 0)
-			(type default)
-		)
-	)
-	(wire
-		(pts
-			(xy 104.14 128.27) (xy 104.14 130.81)
+			(xy 113.03 163.83) (xy 113.03 166.37)
+		)
+		(stroke
+			(width 0)
+			(type default)
+		)
+	)
+	(wire
+		(pts
+			(xy 113.03 161.29) (xy 113.03 163.83)
+		)
+		(stroke
+			(width 0)
+			(type default)
+		)
+	)
+	(wire
+		(pts
+			(xy 113.03 156.21) (xy 113.03 158.75)
+		)
+		(stroke
+			(width 0)
+			(type default)
+		)
+	)
+	(wire
+		(pts
+			(xy 113.03 166.37) (xy 113.03 168.91)
+		)
+		(stroke
+			(width 0)
+			(type default)
+		)
+	)
+	(wire
+		(pts
+			(xy 113.03 171.45) (xy 113.03 173.99)
 		)
 		(stroke
@@
 	(global_label "gnd"
 		(shape input)
-		(at 121.92 151.13 270)
-		(fields_autoplaced yes)
-		(effects
-			(font
-				(size 1.27 1.27)
-			)
-			(justify right)
-		)
-		(property "Intersheetrefs" "${INTERSHEET_REFS}"
-			(at 121.92 157.5622 90)
+		(at 130.81 194.31 270)
+		(fields_autoplaced yes)
+		(effects
+			(font
+				(size 1.27 1.27)
+			)
+			(justify right)
+		)
+		(property "Intersheetrefs" "${INTERSHEET_REFS}"
+			(at 130.81 200.7422 90)
 			(effects
 				(font
@@
 	(symbol
 		(lib_id "MCU_Module:Arduino_Nano_RP2040_Connect")
-		(at 121.92 125.73 0)
+		(at 130.81 168.91 0)
 		(unit 1)
 		(exclude_from_sim no)
@@
 		(fields_autoplaced yes)
 		(property "Reference" "A2"
-			(at 121.92 97.79 0)
+			(at 130.81 140.97 0)
 			(effects
 				(font
@@
 		)
 		(property "Value" "Arduino_Nano_RP2040_Connect"
-			(at 121.92 100.33 0)
+			(at 130.81 143.51 0)
 			(effects
 				(font
@@
 		)
 		(property "Footprint" "Module:Arduino_Nano"
-			(at 135.636 159.766 0)
+			(at 144.526 202.946 0)
 			(effects
 				(font
@@
 		)
 		(property "Datasheet" "https://docs.arduino.cc/resources/datasheets/ABX00053-datasheet.pdf"
-			(at 161.036 157.226 0)
+			(at 169.926 200.406 0)
 			(effects
 				(font
@@
 		)
 		(property "Description" "Arduino Nano board based on the RP2040 microcontroller with a dual-core 133 MHz ARM Cortex-M0+ processor, 264 kB SRAM, and up to 16 MB flash memory. Operates at 3.3V, with 5V Micro USB input and 4-20V VIN. Features Wi-Fi®, Bluetooth® LE, digital and analog pins, and supports SPI, I2C, UART, and PIO. Includes a 6-axis IMU, RGB LED, microphone, and cryptographic chip for secure communication."
-			(at 330.962 154.686 0)
-			(effects
-				(font
+			(at 339.852 197.866 0)
+			(effects
+				(font
